File: 301s/mmp301s-p0_ki9/mmp301s-p0.kicad_sch (KiCad schematic)
At the start: 3 parts, among them Q1 Q_NMOS

Commit message: update sch
Parts:
- removed Q1: Q_NMOS, symbol Device:Q_NMOS
- added Q1: 2SA1488, symbol Device:Q_PNP
- added Q2: 2SC3851, symbol Device:Q_NPN
- added Q3, Q5: 2SA1163, symbol mmp301s-p0:Q_PNP_EBC
- added Q4, Q6: 2SC2713, symbol mmp301s-p0:Q_NPN_EBC
- added R1, R2: R_US, symbol Device:R_US
- added R3, R4, R7, R8: 2R2, symbol Device:R_US
- added R5, R6: 220, symbol Device:R_US
Connections:
- net at U1.21 (~IOUT): now also R2.1
- net at U1.22 (IOUT): now also R1.1
- new net: Q3.B, Q4.B, R7.2
- new net: Q1.C, Q3.C, Q5.C
- new net: Q3.E, Q4.E, R4.1
- new net: R7.1, R8.1
- new net: Q5.B, Q6.B, R8.2
- new net: Q5.E, Q6.E, R3.1
- new net: Q2.B, R3.2, R5.2
- new net: Q2.C, Q4.C, Q6.C
- new net: Q1.E, Q2.E, R5.1, R6.2
- new net: Q1.B, R4.2, R6.1

Commit message: update sch
Parts:
- removed CB1: UL1015_#14_sq2, symbol MMP-H330:CB
- removed Q3, Q5: 2SA1163, symbol mmp301s-p0:Q_PNP_EBC
- removed Q4, Q6: 2SC2713, symbol mmp301s-p0:Q_NPN_EBC
- added C1: C_US, symbol Device:C_US
- added C10, C2, C3, C4, C5, C6, C7, C8, C9: C, symbol mmp301s-p0:C
- added L1: L, symbol mmp301s-p0:L
- added Q10, Q9: 2SA1163, symbol mmp301s-p0:Q_PNP_EBC
- added Q11: 2SC3851, symbol Device:Q_NPN
- added Q12: 2SA1488, symbol Device:Q_PNP
- added Q7, Q8: 2SC2713, symbol mmp301s-p0:Q_NPN_EBC
- added R10, R11, R12, R9: 2R2, symbol Device:R_US
- added R13, R14: 220, symbol Device:R_US
- added R15: 1002, symbol Device:R_US
- added U2: ~, symbol mmp301s-p0:LT1010CN8
- added U3, U4: ~, symbol mmp301s-p0:OPA454
- added U5: LM317, symbol mmp301s-p0:LM317
- R1, R2: value R_US -> 50R0
- R7: value 2R2 -> 50R0
- R8: value 2R2 -> 125R0
- U1: value ~ -> DAC900
Connections:
- net at R7.2: now also U1.18 (FSA)
- net at Q1.C: now also C1.2, U3.4 (V-), U4.4 (V-)
- net at R4.1: now also R3.1, U2.3
- net at R8.1: now also R15.2, U5.3 (VI); no longer R7.1
- net at R8.2: now also U5.1 (ADJ)
- net at Q2.C: now also C1.1, U3.8 (V+), U4.8 (V+)
- net at Q1.E, Q2.E, R5.1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: now also U3.2 (-IN)
- net at U1.11 (Bit11): now also U1.12 (Bit12), U1.13 (Bit13), U1.14 (Bit14), U1.26 (DGND), C2.2, C3.2
- net GNDA: now reaches U1.16 (~INT/EXT)
- net GNDA: now also R1.1, R2.1, R7.1, U1.20 (AGND), C10.2, C4.2, C5.2, C6.2, C7.2, C8.2
- net at U1.17 (REFin): now also C10.1
- net at U1.19 (BW): now also C9.1
- net at U1.21 (~IOUT): now also R2.2, C6.1; no longer R2.1
- net at U1.22 (IOUT): now also R1.2, C7.1, R15.1; no longer R1.1
- net at U1.23 (BYP): now also C8.1
- net at U1.24 (+VA): now also C4.1, C9.2, L1.1
- net +3V3: now reaches U1.27 (+VD)
- net +3V3: now also C2.1, C3.1, C5.1, L1.2
- new net: Q12.B, R12.2, R14.1
- new net: Q11.E, Q12.E, R13.1, R14.2
- new net: R10.1, R9.1
- new net: Q7.B, Q9.B, R9.2
- new net: Q10.C, Q12.C, Q9.C
- new net: Q7.E, Q9.E, R11.1
- new net: U2.8 (INPUT), U3.6 (OUT)
- new net: Q10.B, Q8.B, R10.2
- new net: Q11.B, R11.2, R13.2
- new net: Q10.E, Q8.E, R12.1
- new net: Q11.C, Q7.C, Q8.C
- no-connect marks 0 -> 1
Other:
- note removed: "E"
- note removed: "R"
- note removed: "S"
- moved on the sheet: Q1, Q2, R1, R2, R3, R4, R5, R6, U1

Commit message: 20260525 update
Parts:
- removed C10, C2, C3, C4, C5, C6, C7, C8, C9: C, symbol mmp301s-p0:C
- added C10, C2, C3, C4, C8, C9: C_Small, symbol mmp301s-p0:C_Small
- added C11: C, symbol mmp301s-p0:C
- added C5, C6: 15p, symbol mmp301s-p0:C_Small
- added R16, R17, R18: 1002, symbol Device:R_US
- added R19: 104, symbol mmp301s-p0:R_Small
- added R20: 105, symbol mmp301s-p0:R_Small
- R7: value 50R0 -> 2001
Connections:
- net +3V3: now also C2.1, C4.2
- net GNDA: now also C10.1, C3.1, C4.1, C5.2, C6.2, C8.2
- net at U1.11 (Bit11), U1.12 (Bit12), U1.13 (Bit13)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: now also C2.2
- net at R2.2, U1.21 (~IOUT): now also C5.1
- net at C1.1, Q2.C, U3.8 (V+)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: now also R20.1
- net at C1.2, Q1.C, U3.4 (V-)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: now also U4.1 (ED), R17.1
- net at L1.1, U1.24 (+VA): now also C3.2, C9.2
- net at U1.17 (REFin): now also C10.2
- net at R15.2, R8.1, U5.3 (VI): now also R16.2
- net at R1.2, R15.1, U1.22 (IOUT): now also C6.1
- net at U4.2 (-IN): now also R17.2, R18.2
- net at U4.3 (+IN): now also R16.1
- net at U4.5 (status): now also R20.2
- net at U4.6 (OUT): now also R18.1
- net at U4.7 (E/D): now also R19.2
- net at U1.19 (BW): now also C9.1
- net at U1.23 (BYP): now also C8.1
Other:
- moved on the sheet: C1, L1, Q1, Q2, R1, R2, R3, R4, R5, R6, R7, U2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

Commit message: update 20260608
Parts:
- removed C11: C, symbol mmp301s-p0:C
- removed R16: 1002, symbol Device:R_US
- removed R8: 125R0, symbol Device:R_US
- removed U5: LM317, symbol mmp301s-p0:LM317
- added C7: C, symbol mmp301s-p0:C
- added Q3: BFJ310, symbol mmp301s-p0:Q_NJFET_DGS
- added Q4: C2712, symbol mmp301s-p0:Q_NPN
- added R16: 203, symbol mmp301s-p0:R_Small
- added R21: 1002, symbol Device:R_US
- added R22: 202, symbol mmp301s-p0:R_Small
- added R23: 102, symbol mmp301s-p0:R_Small
- added R24, R25, R8: 103, symbol mmp301s-p0:R_Small
- added RV1: 103VR, symbol mmp301s-p0:RK1631110NTP
- added TP1, TP2, TP3: TP, symbol mmp301s-p0:TB
- added U5: LM358, symbol mmp301s-p0:LM358
- added U6: LM317, symbol mmp301s-p0:LM317
- R18: value 1002 -> 1003
Connections:
- net GNDA: now also C7.2, R16.2, R24.2, U5.4 (V-)
- net at Q1.E, Q2.E, R5.1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: no longer U3.2 (-IN)
- net at R15.2: now also Q4.E, R22.2, R8.1, TP1.1
- net at C6.1, R1.2, R15.1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: now also TP2.1
- net at U4.3 (+IN): now also R8.2
- net at R18.1, U4.6 (OUT): now also TP3.1
- net at R19.1: now also R25.1, U6.2 (VO)
- new net: Q3.3 (S), Q4.B, R22.1
- new net: Q3.1 (D), Q4.C, R21.1, U5.2 (-)
- new net: R24.1, RV1.1, RV1.2, U5.3 (+)
- new net: R23.2, RV1.3
- new net: R16.1, R25.2, U6.1 (ADJ)
- new net: Q3.2 (G), U5.1
- new net +24V: C7.1, R21.2, R23.1, U5.8 (V+), U6.3 (VI)
Other:
- note added: "4.75V"
- note added: "Ix(const.) 1.2mA"
- note added: "Vo=(1+28/10) x Vi =3.8 x Vi x3.8 min 4.788V max 8.588V Center 6.688V 3.8Vp-p x11 min 13.86V max 24.86V Center 19.36V 11.0Vp-p"
- note added: "min 0.06V max 1.06V"
- note added: "min 1.26V max 2.26V"
- moved on the sheet: C1, Q1, Q2, R15, R17, R18, R19, R20, R3, R4, R5, R6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

Commit message: add drive1
Parts:
- removed R3: 2R2, symbol Device:R_US
- removed R5, R6: 220, symbol Device:R_US
- added F1: FUSE-2A, symbol mmp301s-p0:FUSE-axis
- added R26: 203, symbol mmp301s-p0:R_Small
- added R27, R30, R6: 104, symbol mmp301s-p0:R_Small
- added R28: 1002, symbol Device:R_US
- added R29, R3: 103, symbol mmp301s-p0:R_Small
- added R31, R5: 105, symbol mmp301s-p0:R_Small
- added R32: 302, symbol mmp301s-p0:R_Small
- added R33: 331, symbol mmp301s-p0:R_Small
- added R34: 333, symbol mmp301s-p0:R_Small
- added R35: 0R2 2W, symbol Device:R_US
- added TP4: TP, symbol mmp301s-p0:TB
- added U7: ~, symbol mmp301s-p0:OPA454
- R4: value 2R2 -> 0R2 2W
Connections:
- net +24V: now also R26.1
- net at R20.1, U3.8 (V+), U4.8 (V+): now also U2.1 (V+), F1.1, R31.1, R5.1, U7.8 (V+); no longer C1.1, Q2.C
- net at C1.2, R17.1, U3.4 (V-)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: now also R4.1, U2.6 (V-), U3.1 (ED), R27.2, U7.1 (ED), U7.4 (V-); no longer Q1.C
- net at R18.1, TP3.1, U4.6 (OUT): now also R28.2
- net at U2.3: now also Q1.B, Q2.B; no longer R4.1
- net at U2.8 (INPUT): now also U7.6 (OUT); no longer U3.6 (OUT)
- net at Q1.E, Q2.E: now also U7.2 (-IN)
- net at R19.1, R25.1, U6.2 (VO): now also R30.1, R6.1
- net at R4.2: now also Q1.C; no longer Q1.B
- net at U3.2 (-IN): now also R28.1, R33.1
- net at U3.3 (+IN): now also R29.2
- net at U3.5 (status): now also R31.2
- net at U3.7 (E/D): now also R30.2
- net at U5.5 (+): now also R27.1, R32.2
- net at U5.6 (-): now also U5.7, R29.1
- new net: C1.1, F1.2, R35.2
- new net: R5.2, U7.5 (status)
- new net: Q2.C, R35.1
- new net: R3.1, U7.3 (+IN)
- new net: R6.2, U7.7 (E/D)
- new net: R33.2, R34.1
- new net: R3.2, R34.2, TP4.1, U3.6 (OUT)
- new net: R26.2, R32.1
Other:
- added sheet DRIVE_MOCK1 (DRIVE_MOCK1.kicad_sch)
- note added: "19.5V"
- note added: "Ix(const.) 1.2mA min 1.14mA min 2.18mA"
- note added: "Vo=(1+100/10) x Vi =11 x Vi x11 min 13.86V max 24.86V Center 19.36V 11.0Vp-p x3.8 min 4.788V max 8.588V Center 6.688V 3.8Vp-p"
- note added: "Vo=(33.6/10) x Vi =3.33 x Vi x3.32 min 1.6512V max 38.28V Center 6.688V 36.63Vp-p"
- note removed: "2026/04/24 製作時修正内容反映"
- note removed: "Ix(const.) 1.2mA"
- note removed: "Vo=(1+28/10) x Vi =3.8 x Vi x3.8 min 4.788V max 8.588V Center 6.688V 3.8Vp-p x11 min 13.86V max 24.86V Center 19.36V 11.0Vp-p"
- note removed: "注) A. 特記なき接地線は UL1015 AWG18 緑/黄を使用のこと。 B. 特記なきDC線は UL1007 AWG24 (300V 0.2SQ相当)青を使用のこと。 C. 接地は可能な限り1点アースとすること。 D. DC線とAC100V線は極力分離し、幹線と支線の区別をすること。 E. 型式指定、図中指示のないケーブル長は現合とし、極力短く配線すること。 注) 本図型式/メーカー/定格数値は参考とする。"
- moved on the sheet: C1, Q1, Q10, Q11, Q12, Q2, Q7, Q8, Q9, R10, R11, R12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
