File: 301s/mmp301s-p0_ki9/mmp301s-p0.kicad_sch (KiCad schematic)
At the start: 69 parts, among them Q1 2SA1488, Q10 2SA1163, Q11 2SC3851, Q12 2SA1488, Q2 2SC3851, Q3 BFJ310, Q4 C2712, Q7 2SC2713, Q8 2SC2713, Q9 2SA1163, U1 DAC900, U5 LM358, U6 LM317

Commit message: update 20260710
Parts:
- U2: value ~ -> LM1010
- U3, U4, U7: value ~ -> OPA454
Changed lines of the file:
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@@
 			)
 		)
-		(property "Value" "~"
-			(at 356.87 77.3998 0)
+		(property "Value" "LM1010"
+			(at 327.66 87.63 0)
 			(effects
 				(font
@@
 		(dnp no)
 		(property "Reference" "U7"
-			(at 323.85 74.8598 0)
-			(effects
-				(font
-					(size 1.27 1.27)
-				)
-			)
-		)
-		(property "Value" "~"
-			(at 323.85 77.3998 0)
+			(at 314.96 81.28 0)
+			(effects
+				(font
+					(size 1.27 1.27)
+				)
+			)
+		)
+		(property "Value" "OPA454"
+			(at 307.34 87.63 0)
 			(effects
 				(font
@@
 		(on_board yes)
 		(dnp no)
-		(fields_autoplaced yes)
 		(property "Reference" "U3"
-			(at 284.48 77.3998 0)
-			(effects
-				(font
-					(size 1.27 1.27)
-				)
-			)
-		)
-		(property "Value" "~"
-			(at 284.48 79.9398 0)
+			(at 275.59 83.82 0)
+			(effects
+				(font
+					(size 1.27 1.27)
+				)
+			)
+		)
+		(property "Value" "OPA454"
+			(at 267.97 88.9 0)
 			(effects
 				(font
@@
 			)
 		)
-		(property "Value" "~"
+		(property "Value" "OPA454"
 			(at 217.17 77.3998 0)
 			(effects
