File: 301s/301s_drive1/301s_drive1.kicad_pcb (KiCad board)
At the start: 2 copper layers, 95 x 72 mm, 80 parts, among them CN1 B6B-PH, CN2 B12B-PH, CN3 cb_02mail, Q1 TTC3710B, Q13 DTD113ZK, Q14 C2712, Q2 TTA1452B, U1 LM1010, U2 OPA552UA, U3 OPA552UA, U4 LM1010, U5 OPA552UA, U8 LM358DR, U9 DAC900U

Commit message: update 20260713
Parts:
- removed U3: OPA552UA, 301s_drive1:LM358D_SOIC
- Q13: value DTD113ZK -> BFJ310
- R1, R2: value 0R2 2W -> 0R2 1W
- R12, R20: value 273 -> 203
- moved R13 5.00 mm to (114.0, 66.8)
Connections:
- C9 pad 1: /P42V1 -> GND1
- C9 pad 2: GND1 -> /P42V1
- Q14 pad E: Net-(Q14-PadE) -> /WAVE
- R11 pad 1: Net-(U2-+IN) -> Net-(U1-INPUT)
- R11 pad 2: Net-(U3-OUT) -> Net-(U2-OUT)
- R12 pad 1: Net-(U3-Flag) -> Net-(U2-Flag)
- R13 pad 2: Net-(U3-OUT) -> Net-(U2-OUT)
- R14 pad 1: Net-(U3--IN) -> Net-(U2--IN)
- R15 pad 1: /WAVE -> Net-(U5-OUT)
- R15 pad 2: Net-(U3--IN) -> Net-(U2--IN)
- R16 pad 2: Net-(U3-+IN) -> Net-(U2-+IN)
- R21 pad 1: /WAVE -> Net-(U5--IN)
- R21 pad 2: Net-(U5--IN) -> Net-(U5-OUT)
- R22 pad 1: GND1 -> Net-(U5--IN)
- R22 pad 2: Net-(U5--IN) -> GND1
- R23 pad 1: Net-(Q14-PadE) -> /WAVE
- R24 pad 2: Net-(Q14-PadE) -> /WAVE
- R28 pad 1: Net-(Q14-PadE) -> /WAVE
- TP1 pad 1: Net-(U3-OUT) -> Net-(U2-OUT)
- TP5 pad 1: Net-(U3-Flag) -> Net-(U2-Flag)
- TP6 pad 1: /WAVE -> Net-(U5-OUT)
- U2 pad 2: Net-(CN3-Pin_1) -> Net-(U2--IN)
- U2 pad 6: Net-(U1-INPUT) -> Net-(U2-OUT)
- U5 pad 6: /WAVE -> Net-(U5-OUT)
