File: 301s/301s_drive1/301s_drive1.kicad_sch (KiCad schematic)
At the start: 35 parts, among them J1 cb_02mail, J2 Conn_01x06_Pin, Q1 2SC3851, Q2 2SA1488, U1 LM1010, U2 OPA552, U3 OPA552, U4 LM1010

Commit message: update 20260710
Parts:
- removed C4, C7: 106/50V, symbol mmp301s-p0:CAP_POL
- removed C5: 104, symbol mmp301s-p0:C_Small
- removed J2: Conn_01x06_Pin, symbol Connector:Conn_01x06_Pin
- removed R10: 273, symbol mmp301s-p0:R_Small
- removed TP2: CB, symbol mmp301s-p0:CB
- removed U3: OPA552, symbol mmp301s-p0:OPA552
- added C10: 106/50V, 301s_drive1:CP_Radial_D5.0mm_P2.00mm, symbol mmp301s-p0:CAP_POL
- added C12, C14, C15, C16, C18, C20, C7, C8, C9: 104, 301s_drive1:_2012, symbol mmp301s-p0:C_Small
- added C17, C19: 15p, 301s_drive1:_2012, symbol mmp301s-p0:C_Small
- added CN1: B6B-PH, 301s_drive1:B06B-PH, symbol mmp301s-p0:Conn_01x06
- added CN2: B12B-PH, 301s_drive1:B12B-PH, symbol mmp301s-p0:Conn_01x12
- added F2: FUSE-0.5A, 301s_drive1:FUSE0154_, symbol mmp301s-p0:FUSE-axis
- added L1: BLM21BD272SN, 301s_drive1:_2012, symbol mmp301s-p0:L
- added Q13: BFJ310, 301s_drive1:BFJ310, symbol mmp301s-p0:Q_NJFET_DGS
- added Q14: C2712, 301s_drive1:2SC2712, symbol mmp301s-p0:Q_NPN
- added R20, R32, R33, R34, R35, R36, R37, R38, R39, R40, R41, R42: 273, 301s_drive1:R_1608, symbol mmp301s-p0:R_Small
- added R21: 1003, 301s_drive1:R_1608, symbol Device:R_US
- added R22, R25, R28: 1002, 301s_drive1:R_1608, symbol Device:R_US
- added R23: 102, 301s_drive1:R_1608, symbol mmp301s-p0:R_Small
- added R24: 202, 301s_drive1:R_1608, symbol mmp301s-p0:R_Small
- added R26: 362, 301s_drive1:R_1608, symbol mmp301s-p0:R_Small
- added R27: 152, 301s_drive1:R_1608, symbol mmp301s-p0:R_Small
- added R29, R30: 49R9F, 301s_drive1:R_1608, symbol Device:R_US
- added R31: 2001, 301s_drive1:_2012, symbol Device:R_US
- added RV2: 202VR, 301s_drive1:GF063, symbol mmp301s-p0:RK1631110NTP
- added TP7, TP8: CB, 301s_drive1:VIA1.4_inch, symbol mmp301s-p0:CB
- added U5: OPA552UA, 301s_drive1:LM358D_SOIC, symbol mmp301s-p0:OPA552
- added U8: LM358DR, 301s_drive1:LM358D_SOIC, symbol mmp301s-p0:LM358
- added U9: DAC900U, 301s_drive1:DAC900U_SOIC28, symbol mmp301s-p0:DAC904
- C1, C2: footprint (none) -> 301s_drive1:CP_Radial_D5.0mm_P2.00mm
- C3: footprint (none) -> 301s_drive1:_2012
- C6: footprint (none) -> 301s_drive1:CP_Radial_D12.6mm_P5.0mm
- CN3: renamed from J1; footprint (none) -> 301s_drive1:B02B-PH
- F1: footprint (none) -> 301s_drive1:FUSE0154_
- Q1: value 2SC3851 -> TTC3710B; footprint (none) -> 301s_drive1:TO-220L
- Q2: value 2SA1488 -> TTA1452B; footprint (none) -> 301s_drive1:TO-220L
- R1, R2: value 0R2 2W -> 0R2 1W; footprint (none) -> 301s_drive1:R_12
- R11, R12, R13, R14, R16, R17, R18, R19: footprint (none) -> 301s_drive1:R_1608
- R15: value 333 -> 103; footprint (none) -> 301s_drive1:R_1608
- R3: value 101 2W -> 101 1/4W; footprint (none) -> 301s_drive1:R_7.62
- TP1, TP3, TP4, TP5, TP6: footprint (none) -> 301s_drive1:VIA1.4_inch
- U1, U4: footprint (none) -> 301s_drive1:DIP-8_W7.62
- U2: value OPA552 -> OPA552UA; footprint (none) -> 301s_drive1:LM358D_SOIC
Connections:
- net GND1: now also TP4.1, C10.2, C12.2, C14.1, C15.2, C16.1, C17.2, C19.2, C20.1, C7.2, C8.2, C9.2, CN2.12 (Pin_12), R20.2, R22.1, R27.2, R29.1, R30.1, R31.2, U5.1 (V-), U5.4 (V-), U5.5 (V-), U8.4 (V-), U8.5 (+), U9.16 (~INT/EXT), U9.20 (AGND), U9.26 (DGND); no longer TP4.
- net P42V: now also CN1.1 (Pin_1), CN1.2 (Pin_2), F2.1; no longer C1.1, C2.1, C3.1, R19.1, U1.1 (V+), U2.7 (V+), U4.1 (V+)
- net WAVE: now reaches R15.1
- net WAVE: now also TP6.1, R21.1, U5.6 (OUT); no longer TP6.
- net P42V2: now reaches C6.1, F1.2, Q1.C
- net at R11.2, R13.2: now also TP1.1, U2.6 (OUT); no longer TP1.
- net at U1.8 (INPUT): now also R11.1; no longer U2.6 (OUT)
- net at CN3.1 (Pin_1), R1.1, R2.2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: now also TP3.1; no longer TP3., U2.2 (-IN)
- net at R16.2: now also U2.3 (+IN)
- net at U2.8 (Flag): now also R12.1, TP5.1
- net at R14.1, R15.2: now also U2.2 (-IN)
- new net: CN2.1 (Pin_1), R42.2, U9.1 (Bit1)
- new net: CN2.10 (Pin_10), R33.2, U9.10 (Bit10)
- new net: CN2.11 (Pin_11), R32.2, U9.28 (CLK)
- new net: CN2.2 (Pin_2), R41.2, U9.2 (Bit2)
- new net: CN2.3 (Pin_3), R40.2, U9.3 (Bit3)
- new net: CN2.4 (Pin_4), R39.2, U9.4 (Bit4)
- new net: CN2.5 (Pin_5), R38.2, U9.5 (Bit5)
- new net: CN2.6 (Pin_6), R37.2, U9.6 (Bit6)
- new net: CN2.7 (Pin_7), R36.2, U9.7 (Bit7)
- new net: CN2.8 (Pin_8), R35.2, U9.8 (Bit8)
- new net: CN2.9 (Pin_9), R34.2, U9.9 (Bit9)
- new net: U1.4 (NC), U1.5 (NC), U1.7 (NC)
- new net: R21.2, R22.2, U5.2 (-IN)
- new net: Q13.D, Q14.C, R25.1, U8.2 (-)
- new net: Q13.G, U8.1
- new net: Q13.S, Q14.B, R24.1
- new net: C18.1, U9.19 (BW)
- new net: Q14.E, R23.1, R24.2, R28.1
- new net: C19.1, R28.2, R29.2, TP7.1, U9.22 (IOUT)
- new net: R26.2, RV2.3
- new net: C17.1, R30.2, U9.21 (~IOUT)
- new net: R31.1, U9.18 (FSA)
- new net: R20.1, U5.8 (Flag)
- new net: R27.1, RV2.1, RV2.2, TP8.1, U8.3 (+)
- new net: U8.6 (-), U8.7
- new net: C16.2, U9.17 (REFin)
- new net: R23.2, U5.3 (+IN)
- new net: C15.1, U9.23 (BYP)
- new net: U4.4 (NC), U4.5 (NC), U4.7 (NC)
- new net +3V3: C12.1, C20.2, CN1.4 (Pin_4), L1.2, R32.1, R33.1, R34.1, R35.1, R36.1, R37.1, R38.1, R39.1, R40.1, R41.1, R42.1, U9.27 (+VD)
- new net +5V: C8.1, CN1.3 (Pin_3), R25.2, R26.1, U8.8 (V+)
- new net 3R3A: C14.2, C18.2, L1.1, U9.24 (+VA)
- new net GND: CN1.5 (Pin_5), CN1.6 (Pin_6)
- new net P42V1: C1.1, C10.1, C2.1, C3.1, C7.1, C9.1, F2.2, R19.1, U1.1 (V+), U2.7 (V+), U4.1 (V+), U5.7 (V+)
- no-connect marks 3 -> 10
Other:
- note added: "Ix 1.2mA"
- note added: "Step1 出力段評価 5Pコネクタ 1,2-42V 3-Sig 4,5-GND TP1に104プルダウン"
- note added: "Vo=(1+100/10) x Vi =11 x Vi x11 min 13.86V max 24.86V Center 19.36V 11.0Vp-p x3.8 min 4.788V max 8.588V Center 6.688V 3.8Vp-p"
- note added: "Vo=(33.6/10) x Vi =3.33 x Vi x3.32 min 1.6512V max 38.28V Center 6.688V 36.63Vp-p"
- note added: "min 0.06V max 1.06V"
- note added: "min 1.05V max 1.47V"
- note added: "min 1.26V max 2.26V"
- note removed: "TP1: Vo=(33.6/10) x Vi =3.33 x Vi x3.32 min 1.6512V max 38.28V Center 6.688V 36.63Vp-p"
- moved on the sheet: C1, C2, C3, C6, CN3, F1, Q1, Q2, R1, R11, R12, R13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

Commit message: update 20260713
Parts:
- removed R21: 1003, 301s_drive1:R_1608, symbol Device:R_US
- removed R22: 1002, 301s_drive1:R_1608, symbol Device:R_US
- added R21: 1003, 301s_drive1:R_1608, symbol mmp301s-p0:R_Small
- added R22: 1002, 301s_drive1:R_1608, symbol mmp301s-p0:R_Small
- R12, R20: value 273 -> 203
Connections:
- net GND1: now also C9.1, R22.2; no longer C9.2
- net P42V1: now also C9.2; no longer C9.1
- net WAVE: now also Q14.E, R23.1, R24.2, R28.1; no longer R15.1, TP6.1, U5.6 (OUT)
- net at U5.2 (-IN): now also R21.1, R22.1
- new net: R15.1, R21.2, TP6.1, U5.6 (OUT)
Other:
- note added: "19.5V"
- note added: "Vo=(1+100/10) x Vi =11 x Vi x11 min 13.86V max 24.86V Center 19.36V 11.0Vp-p"
- note removed: "TP6: Vo=(1+100/10) x Vi =11 x Vi x11 min 13.86V max 24.86V Center 19.36V 11.0Vp-p x3.8 min 4.788V max 8.588V Center 6.688V 3.8Vp-p"
- note removed: "Vo=(1+100/10) x Vi =11 x Vi x11 min 13.86V max 24.86V Center 19.36V 11.0Vp-p x3.8 min 4.788V max 8.588V Center 6.688V 3.8Vp-p"
- moved on the sheet: C10, C7, C9, CN1, F1, F2, R15, R17, R18, R19, R20, R23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

Commit message: 2026/08/05 update 3
Connections:
- net at R16.1: now also R21.2, U5.6 (OUT); no longer U4.3
- net at R14.1, R15.2, U2.2 (-IN): now also TP6.1
- new net: R15.1, U4.3
Other:
- note added: "19.0V"
- note added: "2028/08/05 U2を反転増幅で基本動作できた。U2を非反転3.33倍増幅回路にしないと DAC出力のデジタルデータを反転しなければならないので、非反転増幅回路を追加確認する。"
- note added: "Vo=(33.6/10) x Vi =3.33 x Vi x3.32 min 1.88V max 38.51V 36.63Vp-p"
- note removed: "19.5V"
- note removed: "Vo=(33.6/10) x Vi =3.33 x Vi x3.32 min 1.6512V max 38.28V Center 6.688V 36.63Vp-p"
- moved on the sheet: R15, R16, TP6
Changed lines of the file:
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@@
 	(paper "A4")
 	(title_block
-		(date "2026-07-13")
+		(date "2026-08-05")
 		(comment 1 "S301-100-0")
 		(comment 2 "DRIVE1")
@@
 		)
 	)
+	(text "2028/08/05\nU2を反転増幅で基本動作できた。U2を非反転3.33倍増幅回路にしないと\nDAC出力のデジタルデータを反転しなければならないので、非反転増幅回路を追加確認する。"
+		(exclude_from_sim no)
+		(at 215.9 144.78 0)
+		(effects
+			(font
+				(size 1.27 1.27)
+			)
+			(justify left top)
+		)
+	)
 	(text "Step1　出力段評価\n	5Pコネクタ 1,2-42V 3-Sig 4,5-GND\n	TP1に104プルダウン"
 		(exclude_from_sim no)
@@
 		)
 	)
-	(text "19.5V"
+	(text "19.0V"
 		(exclude_from_sim no)
-		(at 130.81 82.55 0)
+		(at 133.35 82.55 0)
 		(effects
 			(font
@@
 		)
 	)
-	(text "\nVo=(33.6/10) x Vi\n  =3.33 x Vi\nx3.32\n  min 1.6512V\n  max 38.28V\n  Center 6.688V\n  36.63Vp-p"
+	(text "\nVo=(33.6/10) x Vi\n  =3.33 x Vi\nx3.32\n  min 1.88V\n  max 38.51V\n  36.63Vp-p"
 		(exclude_from_sim no)
 		(at 161.29 85.09 0)
@@
 	)
 	(junction
+		(at 129.54 67.31)
+		(diameter 0)
+		(color 0 0 0 0)
+	)
+	(junction
 		(at 129.54 147.32)
 		(diameter 0)
@@
 	)
 	(junction
+		(at 97.79 69.85)
+		(diameter 0)
+		(color 0 0 0 0)
+	)
+	(junction
 		(at 123.19 190.5)
 		(diameter 0)
@@
 	)
 	(junction
-		(at 119.38 57.15)
-		(diameter 0)
-		(color 0 0 0 0)
-	)
-	(junction
 		(at 152.4 93.98)
 		(diameter 0)
@@
 	)
 	(junction
-		(at 97.79 57.15)
-		(diameter 0)
-		(color 0 0 0 0)
-	)
-	(junction
 		(at 80.01 121.92)
 		(diameter 0)
@@
 	(wire
 		(pts
-			(xy 97.79 57.15) (xy 87.63 57.15)
+			(xy 129.54 80.01) (xy 129.54 82.55)
 		)
 		(stroke
@@
 	(wire
 		(pts
-			(xy 114.3 182.88) (xy 116.84 182.88)
+			(xy 97.79 57.15) (xy 87.63 57.15)
 		)
 		(stroke
@@
 	(wire
 		(pts
-			(xy 123.19 190.5) (xy 129.54 190.5)
+			(xy 114.3 182.88) (xy 116.84 182.88)
 		)
 		(stroke
@@
 	(wire
 		(pts
-			(xy 44.45 31.75) (xy 57.15 31.75)
+			(xy 123.19 190.5) (xy 129.54 190.5)
 		)
 		(stroke
@@
 	(wire
 		(pts
-			(xy 69.85 116.84) (xy 69.85 104.14)
+			(xy 44.45 31.75) (xy 57.15 31.75)
 		)
 		(stroke
@@
 	(wire
 		(pts
-			(xy 127 82.55) (xy 127 72.39)
+			(xy 69.85 116.84) (xy 69.85 104.14)
 		)
 		(stroke
@@
 	(wire
 		(pts
-			(xy 124.46 82.55) (xy 127 82.55)
+			(xy 124.46 82.55) (xy 129.54 82.55)
 		)
 		(stroke
@@
 	(wire
 		(pts
+			(xy 129.54 74.93) (xy 129.54 67.31)
+		)
+		(stroke
+			(width 0)
+			(type default)
+		)
+	)
+	(wire
+		(pts
 			(xy 102.87 52.07) (xy 102.87 82.55)
 		)
@@
 	(wire
 		(pts
-			(xy 134.62 72.39) (xy 142.24 72.39)
+			(xy 124.46 72.39) (xy 142.24 72.39)
 		)
 		(stroke
@@
 	(wire
 		(pts
-			(xy 127 72.39) (xy 129.54 72.39)
+			(xy 97.79 69.85) (xy 119.38 72.39)
 		)
 		(stroke
@@
 	(wire
 		(pts
-			(xy 97.79 57.15) (xy 119.38 57.15)
-		)
-		(stroke
-			(width 0)
-			(type default)
-		)
-	)
-	(wire
-		(pts
-			(xy 119.38 54.61) (xy 119.38 57.15)
-		)
-		(stroke
-			(width 0)
-			(type default)
-		)
-	)
-	(wire
-		(pts
 			(xy 152.4 80.01) (xy 152.4 83.82)
 		)
@@
 	(wire
 		(pts
-			(xy 119.38 57.15) (xy 121.92 57.15)
-		)
-		(stroke
-			(width 0)
-			(type default)
-		)
-	)
-	(wire
-		(pts
 			(xy 224.79 85.09) (xy 224.79 93.98)
 		)
@@
 	(symbol
 		(lib_id "mmp301s-p0:R_Small")
-		(at 132.08 72.39 90)
+		(at 121.92 72.39 90)
 		(unit 1)
 		(exclude_from_sim no)
@@
 		(dnp no)
 		(property "Reference" "R16"
-			(at 130.175 69.215 90)
+			(at 120.015 69.215 90)
 			(effects
 				(font
@@
 		)
 		(property "Value" "102"
-			(at 130.175 71.12 90)
+			(at 120.015 71.12 90)
 			(effects
 				(font
@@
 		)
 		(property "Footprint" "301s_drive1:R_1608"
-			(at 132.08 72.39 0)
+			(at 121.92 72.39 0)
 			(effects
 				(font
@@
 		)
 		(property "Datasheet" ""
-			(at 132.08 72.39 0)
+			(at 121.92 72.39 0)
 			(effects
 				(font
@@
 		)
 		(property "Description" ""
-			(at 132.08 72.39 0)
+			(at 121.92 72.39 0)
 			(effects
 				(font
@@
 	(symbol
 		(lib_id "mmp301s-p0:R_Small")
-		(at 124.46 57.15 90)
+		(at 129.54 77.47 180)
 		(unit 1)
 		(exclude_from_sim no)
@@
 		(dnp no)
 		(property "Reference" "R15"
-			(at 122.555 53.975 90)
+			(at 126.365 79.375 90)
 			(effects
 				(font
@@
 		)
 		(property "Value" "103"
-			(at 122.555 55.88 90)
+			(at 128.27 79.375 90)
 			(effects
 				(font
@@
 		)
 		(property "Footprint" "301s_drive1:R_1608"
-			(at 124.46 57.15 0)
+			(at 129.54 77.47 0)
 			(effects
 				(font
@@
 		)
 		(property "Datasheet" ""
-			(at 124.46 57.15 0)
+			(at 129.54 77.47 0)
 			(effects
 				(font
@@
 		)
 		(property "Description" ""
-			(at 124.46 57.15 0)
+			(at 129.54 77.47 0)
 			(effects
 				(font
@@
 	(symbol
 		(lib_id "mmp301s-p0:CB")
-		(at 119.38 54.61 0)
+		(at 127 57.15 0)
 		(unit 1)
 		(exclude_from_sim no)
@@
 		(dnp no)
 		(property "Reference" "TP6"
-			(at 118.11 53.34 0)
+			(at 125.73 55.88 0)
 			(effects
 				(font
@@
 		)
 		(property "Value" "CB"
-			(at 119.38 50.8 0)
+			(at 127 53.34 0)
 			(effects
 				(font
@@
 		)
 		(property "Footprint" "301s_drive1:VIA1.4_inch"
-			(at 119.38 53.34 0)
+			(at 127 55.88 0)
 			(effects
 				(font
@@
 		)
 		(property "Datasheet" ""
-			(at 119.38 53.34 0)
+			(at 127 55.88 0)
 			(effects
 				(font
@@
 		)
 		(property "Description" ""
-			(at 119.38 54.61 0)
+			(at 127 57.15 0)
 			(effects
 				(font
